File: PCB design/EIinUtilityDisplay.kicad_sch (KiCad schematic)
At the start: 70 parts, among them J1 USB_C_Receptacle_USB2.0_16P, J2 Conn_01x12_Pin, SW0 Q, SW1 W, SW10 A, SW11 S, SW12 D, SW13 F, SW14 G, SW15 H, SW16 J, SW17 K, SW18 L, SW19 " ', SW2 E, SW20 Z, SW21 X, SW22 C, SW23 V, SW24 B, SW25 N, SW26 M, SW27 , -, SW28 . +, SW29 ? /, SW3 R, SW31 TAB, SW32 CAPS, SW33 SHIFT, SW34 CTRL, SW35 SPACE, SW36 ALT, SW37 [ }, SW38 ] }, SW39 ENTER, SW4 T, SW40 0, SW41 1, SW42 2, SW43 3, SW44 4, SW45 5, SW46 6, SW47 7, SW48 8, SW49 9, SW5 Y, SW51 SW_Push_Dual, SW6 U, SW7 I, SW8 O, SW9 P, U1 TCA8418RTWR, U2 MCP73831-2-OT

Commit message: added ESP32
Parts:
- added BT1: Battery, symbol Device:Battery
- added C4: 22μF, symbol Device:C_Polarized
- added C5: 10μF, symbol Device:C_Polarized
- added C6, C7: 1μF, symbol Device:C
- added D3: 1N4148W, symbol Device:D
- added Q1: IRLML5103TRPBF, IRLML5103TRPBF:SOT95P237X112-3N, symbol irlml6302trpbf:IRLML5103TRPBF
- added R11, R12: 10k, symbol Device:R
- added SW50: Z + Ctrl, symbol Switch:SW_Push_Dual
- added SW51: Y + Ctrl, symbol Switch:SW_Push_Dual
- added SW52, SW53: SW_SPST, symbol Switch:SW_SPST
- added U3: ADP3338AKCZ-3.3-RL, ADP3338AKCZ-3.3-RL:SOT230P700X180-4N, symbol regulator:ADP3338AKCZ-3.3-RL
- added U4: ESP32-S3-WROOM-1, RF_Module:ESP32-S3-WROOM-1, symbol RF_Module:ESP32-S3-WROOM-1
- SW-PWR: renamed from SW51; value SW_Push_Dual -> On/Off
Connections:
- net +3.3V: now also C4.1, R11.1, U3.2 (OUT), U3.4 (OUT), U4.2 (3V3)
- net BAT+: now also BT1.1 (+), Q1.3
- net GND: now also BT1.2 (-), C4.2, C5.2, C6.2, C7.1, SW52.2 (B), SW53.2 (B), U3.1 (GND), U4.1 (GND), U4.40 (GND), U4.41 (GND)
- net battMeas: now also U4.6 (IO6)
- net col0: now also SW50.1
- net col4: now also SW50.3, SW51.3
- net col5: now also SW51.1
- net pwrBtn: now also U4.31 (IO38)
- net row0: now also SW51.2
- net row2: now also SW50.2
- net row3: now also SW50.4, SW51.4
- net usb5V: now also D3.2 (A), Q1.1
- net usbD+: now also U4.14 (USB_D+)
- net usbD-: now also U4.13 (USB_D-)
- new net: R12.2, SW53.1 (A)
- new net: C6.1, R11.2
- new net: C5.1, D3.1 (K), Q1.2, U3.3 (IN)
- new net BOOT: R12.1, U4.27 (IO0)
- new net BUSY: U4.30 (IO37)
- new net CS: U4.38 (IO2)
- new net D/C: U4.23 (IO21)
- new net EN: C7.2, SW52.1 (A), U4.3 (EN)
- new net I2C-SCL: U4.28 (IO35)
- new net I2C-SDA: U4.29 (IO36)
- new net INT: U4.12 (IO8)
- new net MagSense: U4.15 (IO3)
- new net RESET: U4.9 (IO16)
- new net SPI-MISO: U4.21 (IO13)
- new net SPI-MOSI: U4.19 (IO11)
- new net SPI-SCK: U4.20 (IO12)
- no-connect marks 8 -> 14
Other:
- moved on the sheet: C1, C2, C3, D1, D2, J1, J2, R1, R10, R2, R3, R4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
